Commit message: feat: Add 7-DOF linear track, new STLs, and 3D Coverage Path Planning executor

File: ros2_ws/src/irb2600_description/urdf/irb2600.urdf.xacro (robot description, xacro)
@@ -1,20 +1,6 @@
 <?xml version="1.0"?>
 <robot name="abb_irb2600_coating_cell" xmlns:xacro="http://ros.org/wiki/xacro">
-  <!--
-    ROS 2 equivalent of RAMEL-ESPOL/IRB2600-ABB irb2600_description/urdf/irb2600_main.xacro,
-    trimmed to what the DIMECA coating-cell digital prototype needs: the bare robot on
-    its pedestal plus the spray-nozzle end effector. Table/wall/other tool variants from
-    the original file were dropped; the target structure and obstacle are NOT part of
-    this URDF (they are inserted as collision objects into the MoveIt planning scene at
-    runtime by irb2600_coating_cell, since the report treats the obstacle as dynamic).
-  -->
   <link name="world"/>
-  <!--
-    materials.xacro is included exactly once, here, before anything that
-    uses xacro:material_abb_orange. xacro does not deduplicate repeated
-    xacro:include of the same file, and urdfdom rejects a <material> name
-    that is defined (i.e. with a color/texture child) more than once, so
-    irb2600_macro.xacro and spray_nozzle.xacro must NOT also include it.
-  -->
+  <!-- Included macros -->
   <xacro:include filename="$(find irb2600_description)/urdf/materials.xacro"/>
   <xacro:include filename="$(find irb2600_description)/urdf/irb2600_macro.xacro"/>
@@ -22,4 +8,69 @@
   <xacro:include filename="$(find irb2600_description)/urdf/spray_nozzle.xacro"/>
   <xacro:include filename="$(find irb2600_description)/urdf/ros2_control.xacro"/>
+  <!-- Track and Platform Links -->
+  <link name="track_link">
+    <visual>
+      <origin xyz="0 0 0" rpy="0 0 0"/>
+      <geometry>
+        <mesh filename="package://irb2600_coating_cell/meshes/Riel.stl" scale="0.001 0.001 0.001"/>
+      </geometry>
+      <material name="pedestal_coral"/>
+    </visual>
+    <collision>
+      <origin xyz="0 0 0" rpy="0 0 0"/>
+      <geometry>
+        <mesh filename="package://irb2600_coating_cell/meshes/Riel.stl" scale="0.001 0.001 0.001"/>
+      </geometry>
+    </collision>
+    <inertial>
+      <origin xyz="0 0 0" rpy="0 0 0"/>
+      <mass value="500.0"/>
+      <inertia ixx="1.0" ixy="0.0" ixz="0.0" iyy="1.0" iyz="0.0" izz="1.0"/>
+    </inertial>
+  </link>
+  <link name="platform_link">
+    <visual>
+      <origin xyz="0 0 0" rpy="0 0 0"/>
+      <geometry>
+        <mesh filename="package://irb2600_coating_cell/meshes/PlataformaRiel.STL" scale="0.001 0.001 0.001"/>
+      </geometry>
+      <material name="pedestal_coral"/>
+    </visual>
+    <collision>
+      <origin xyz="0 0 0" rpy="0 0 0"/>
+      <geometry>
+        <mesh filename="package://irb2600_coating_cell/meshes/PlataformaRiel.STL" scale="0.001 0.001 0.001"/>
+      </geometry>
+    </collision>
+    <inertial>
+      <origin xyz="0 0 0" rpy="0 0 0"/>
+      <mass value="50.0"/>
+      <inertia ixx="0.1" ixy="0.0" ixz="0.0" iyy="0.1" iyz="0.0" izz="0.1"/>
+    </inertial>
+  </link>
+  <!-- Joints connecting World -> Track -> Platform -->
+  <!-- Assume the track lies flat on the ground. We might need to adjust RPY if the STL Z is the length -->
+  <!-- The user said Z is 8610, which means the track is aligned with Z. If it should be horizontal (Y axis), we rotate it. -->
+  <!-- Let's keep it as is first, we can view it in RViz later. -->
+  <joint name="world_to_track_joint" type="fixed">
+    <parent link="world"/>
+    <child link="track_link"/>
+    <!-- Rotate so the 8.6m Z-axis of the STL becomes the Y-axis of the world -->
+    <origin xyz="0 0 0" rpy="1.5708 0 0"/>
+  </joint>
+  <!-- Prismatic joint for the linear track -->
+  <joint name="track_prismatic_joint" type="prismatic">
+    <parent link="track_link"/>
+    <child link="platform_link"/>
+    <!-- The track slides along the STL's Z axis (which is now world Y) -->
+    <axis xyz="0 0 1"/>
+    <origin xyz="0 0 0" rpy="0 0 0"/>
+    <!-- Limits: from 0 to roughly the length of the track minus platform -->
+    <limit lower="0.0" upper="4.5" effort="1000.0" velocity="0.5"/>
+  </joint>
+  <!-- Mount the robot's base_mesh to the platform -->
+  <!-- In robot_base.xacro, base_mesh attaches to 'world'. We will change that file later so it attaches to 'platform_link'. -->
+  <!-- Or we can just not include robot_base.xacro and do it here? robot_base.xacro has base_mesh_joint. -->
+  <!-- Load robot -->
   <xacro:abb_irb2600 prefix=""/>
   <xacro:abb_irb2600_ros2_control prefix=""/>

File: ros2_ws/src/irb2600_description/urdf/robot_base.xacro (robot description, xacro)
@@ -26,7 +26,9 @@
   </link>
   <joint name="base_mesh_joint" type="fixed">
-    <parent link="world"/>
+    <parent link="platform_link"/>
     <child link="base_mesh"/>
-    <origin xyz="0 0 0.209" rpy="0 0 0"/>
+    <!-- The platform STL Z size is ~4.18m but that's probably length, let's assume thickness is much smaller. We'll adjust Z offset if needed later. -->
+    <!-- Let's put Z=0.1 for now until we can visualize it. -->
+    <origin xyz="0 0 0.1" rpy="0 0 0"/>
   </joint>
   <joint name="base_robot_joint" type="fixed">

File: ros2_ws/src/irb2600_description/urdf/ros2_control.xacro (robot description, xacro)
@@ -16,4 +16,9 @@
         <plugin>mock_components/GenericSystem</plugin>
       </hardware>
+      <joint name="track_prismatic_joint">
+        <command_interface name="position"/>
+        <state_interface name="position"/>
+        <state_interface name="velocity"/>
+      </joint>
       <joint name="${prefix}joint_1">
         <command_interface name="position"/>

File: ros2_ws/src/irb2600_description/urdf/spray_nozzle.xacro (robot description, xacro)
@@ -35,5 +35,5 @@
       <origin xyz="0 0 0" rpy="0 0 0"/>
       <geometry>
-        <mesh filename="package://irb2600_description/meshes/supports/spray_nozzle.STL"/>
+        <mesh filename="package://irb2600_coating_cell/meshes/CobraPaintTool.STL" scale="0.001 0.001 0.001"/>
       </geometry>
       <xacro:material_abb_orange/>
@@ -42,5 +42,5 @@
       <origin xyz="0 0 0" rpy="0 0 0"/>
       <geometry>
-        <mesh filename="package://irb2600_description/meshes/supports/spray_nozzle.STL"/>
+        <mesh filename="package://irb2600_coating_cell/meshes/CobraPaintTool.STL" scale="0.001 0.001 0.001"/>
       </geometry>
     </collision>

Commit message: feat: Add target panel directly to URDF to guarantee visibility in RViz without relying on python markers

File: ros2_ws/src/irb2600_description/urdf/irb2600.urdf.xacro (robot description, xacro)
@@ -72,4 +72,27 @@
   <!-- In robot_base.xacro, base_mesh attaches to 'world'. We will change that file later so it attaches to 'platform_link'. -->
   <!-- Or we can just not include robot_base.xacro and do it here? robot_base.xacro has base_mesh_joint. -->
+  <!-- Hardcoded Target Panel for guaranteed visibility in RViz without DDS issues -->
+  <link name="target_panel">
+    <visual>
+      <origin xyz="0 0 0" rpy="0 0 0"/>
+      <geometry>
+        <box size="0.05 5.0 2.0"/>
+      </geometry>
+      <material name="panel_blue">
+        <color rgba="0.2 0.5 1.0 1.0"/>
+      </material>
+    </visual>
+    <collision>
+      <origin xyz="0 0 0" rpy="0 0 0"/>
+      <geometry>
+        <box size="0.05 5.0 2.0"/>
+      </geometry>
+    </collision>
+  </link>
+  <joint name="world_to_panel" type="fixed">
+    <parent link="world"/>
+    <child link="target_panel"/>
+    <origin xyz="1.5 -4.5 1.5" rpy="0 0 0"/>
+  </joint>
   <!-- Load robot -->
   <xacro:abb_irb2600 prefix=""/>

Commit message: feat: Visual paint simulation. Panel is now white, and a trail of blue paint splatters is drawn in RViz along the executed trajectory

File: ros2_ws/src/irb2600_description/urdf/irb2600.urdf.xacro (robot description, xacro)
@@ -79,6 +79,6 @@
         <box size="0.05 5.0 2.0"/>
       </geometry>
-      <material name="panel_blue">
-        <color rgba="0.2 0.5 1.0 1.0"/>
+      <material name="panel_white">
+        <color rgba="1.0 1.0 1.0 1.0"/>
       </material>
     </visual>

Commit message: feat: Replace basic grid generator with advanced 3D mesh coverage path planner using trimesh raycasting and precise surface normals

File: ros2_ws/src/irb2600_description/urdf/irb2600.urdf.xacro (robot description, xacro)
@@ -75,7 +75,7 @@
   <link name="target_panel">
     <visual>
-      <origin xyz="0 0 0" rpy="0 0 0"/>
+      <origin xyz="0 0 0" rpy="1.5708 0 0"/>
       <geometry>
-        <box size="0.05 5.0 2.0"/>
+        <mesh filename="package://irb2600_coating_cell/meshes/wavy_panel.stl"/>
       </geometry>
       <material name="panel_white">
@@ -84,7 +84,7 @@
     </visual>
     <collision>
-      <origin xyz="0 0 0" rpy="0 0 0"/>
+      <origin xyz="0 0 0" rpy="1.5708 0 0"/>
       <geometry>
-        <box size="0.05 5.0 2.0"/>
+        <mesh filename="package://irb2600_coating_cell/meshes/wavy_panel.stl"/>
       </geometry>
     </collision>

Commit message: fix: Declare mesh_file parameter and move panel to avoid track collision

File: ros2_ws/src/irb2600_description/urdf/irb2600.urdf.xacro (robot description, xacro)
@@ -93,5 +93,5 @@
     <parent link="world"/>
     <child link="target_panel"/>
-    <origin xyz="1.5 -4.5 1.5" rpy="0 0 0"/>
+    <origin xyz="2.0 2.0 1.5" rpy="0 0 0"/>
   </joint>
   <!-- Load robot -->

Commit message: fix: Regenerate wavy panel STL with correct orientation and remove arbitrary 90deg rotations that caused out-of-bounds Z reach issues in IK solver

File: ros2_ws/src/irb2600_description/urdf/irb2600.urdf.xacro (robot description, xacro)
@@ -75,5 +75,5 @@
   <link name="target_panel">
     <visual>
-      <origin xyz="0 0 0" rpy="1.5708 0 0"/>
+      <origin xyz="0 0 0" rpy="0 0 0"/>
       <geometry>
         <mesh filename="package://irb2600_coating_cell/meshes/wavy_panel.stl"/>
@@ -84,5 +84,5 @@
     </visual>
     <collision>
-      <origin xyz="0 0 0" rpy="1.5708 0 0"/>
+      <origin xyz="0 0 0" rpy="0 0 0"/>
       <geometry>
         <mesh filename="package://irb2600_coating_cell/meshes/wavy_panel.stl"/>

Commit message: fix: Move panel back to X=1.5 and precisely to Y=-2.25 to stay within the robot's reachable kinematic envelope

File: ros2_ws/src/irb2600_description/urdf/irb2600.urdf.xacro (robot description, xacro)
@@ -93,5 +93,5 @@
     <parent link="world"/>
     <child link="target_panel"/>
-    <origin xyz="2.0 2.0 1.5" rpy="0 0 0"/>
+    <origin xyz="1.5 -2.25 1.5" rpy="0 0 0"/>
   </joint>
   <!-- Load robot -->

Commit message: feat: Replace wavy panel with a compact 3D industrial tank object for real-world coverage path planning demonstration

File: ros2_ws/src/irb2600_description/urdf/irb2600.urdf.xacro (robot description, xacro)
@@ -77,5 +77,5 @@
       <origin xyz="0 0 0" rpy="0 0 0"/>
       <geometry>
-        <mesh filename="package://irb2600_coating_cell/meshes/wavy_panel.stl"/>
+        <mesh filename="package://irb2600_coating_cell/meshes/tank.stl"/>
       </geometry>
       <material name="panel_white">
@@ -86,12 +86,13 @@
       <origin xyz="0 0 0" rpy="0 0 0"/>
       <geometry>
-        <mesh filename="package://irb2600_coating_cell/meshes/wavy_panel.stl"/>
+        <mesh filename="package://irb2600_coating_cell/meshes/tank.stl"/>
       </geometry>
     </collision>
   </link>
+  <!-- Mount target panel to world at the center of the track reach -->
   <joint name="world_to_panel" type="fixed">
     <parent link="world"/>
     <child link="target_panel"/>
-    <origin xyz="1.5 -2.25 1.5" rpy="0 0 0"/>
+    <origin xyz="1.5 -2.25 1.0" rpy="0 0 0"/>
   </joint>
   <!-- Load robot -->

Commit message: fix: Adjust X coordinate of tank to 2.4 to account for track platform width and offset base, placing it at optimal 1.2m reach distance

File: ros2_ws/src/irb2600_description/urdf/irb2600.urdf.xacro (robot description, xacro)
@@ -94,5 +94,5 @@
     <parent link="world"/>
     <child link="target_panel"/>
-    <origin xyz="1.5 -2.25 1.0" rpy="0 0 0"/>
+    <origin xyz="2.4 -2.25 1.0" rpy="0 0 0"/>
   </joint>
   <!-- Load robot -->

Commit message: feat: Rotate track 180 degrees to shield cables behind the robot, while perfectly preserving the robot's world-frame facing and workspace reachability towards the workpiece

File: ros2_ws/src/irb2600_description/urdf/irb2600.urdf.xacro (robot description, xacro)
@@ -56,6 +56,6 @@
     <parent link="world"/>
     <child link="track_link"/>
-    <!-- Rotate so the 8.6m Z-axis of the STL becomes the Y-axis of the world -->
-    <origin xyz="0 0 0" rpy="1.5708 0 0"/>
+    <!-- Rotate 180 around Z to put cables on the back. Shift Y by -8.6 to keep track in the same space -->
+    <origin xyz="0 -8.6 0" rpy="1.5708 0 3.14159265359"/>
   </joint>
   <!-- Prismatic joint for the linear track -->
@@ -94,5 +94,5 @@
     <parent link="world"/>
     <child link="target_panel"/>
-    <origin xyz="2.4 -2.25 1.0" rpy="0 0 0"/>
+    <origin xyz="1.1 -4.85 1.0" rpy="0 0 0"/>
   </joint>
   <!-- Load robot -->

File: ros2_ws/src/irb2600_description/urdf/robot_base.xacro (robot description, xacro)
@@ -28,6 +28,6 @@
     <parent link="platform_link"/>
     <child link="base_mesh"/>
-    <!-- The platform's Y axis points UP (World Z), so we offset in Y to place it on top, and rotate -90 deg around X to make the robot's Z point UP. -->
-    <origin xyz="0.65 0.6 1.5" rpy="-1.5708 0 0"/>
+    <!-- Add 180 yaw (-3.14159) to keep robot facing World +X despite platform rotation -->
+    <origin xyz="0.65 0.6 1.5" rpy="1.5708 0 3.14159265359"/>
   </joint>
   <joint name="base_robot_joint" type="fixed">

Commit message: feat: Revert rail flip, realign global origin, and switch to a 4m x 2m curved surface panel

File: ros2_ws/src/irb2600_description/urdf/irb2600.urdf.xacro (robot description, xacro)
@@ -56,6 +56,5 @@
     <parent link="world"/>
     <child link="track_link"/>
-    <!-- Rotate 180 around Z to put cables on the back. Shift Y by -8.6 to keep track in the same space -->
-    <origin xyz="0 -8.6 0" rpy="1.5708 0 3.14159265359"/>
+    <origin xyz="0 0 0" rpy="1.5708 0 0"/>
   </joint>
   <!-- Prismatic joint for the linear track -->
@@ -63,9 +62,10 @@
     <parent link="track_link"/>
     <child link="platform_link"/>
-    <!-- The track slides along the STL's Z axis (which is now world Y) -->
+    <!-- The STL's Z-axis corresponds to the length of the track -->
     <axis xyz="0 0 1"/>
-    <origin xyz="0 0 0" rpy="0 0 0"/>
-    <!-- Limits: from 0 to roughly the length of the track minus platform -->
-    <limit lower="0.0" upper="4.5" effort="1000.0" velocity="0.5"/>
+    <!-- The physical track limits. Since we rotated it, +Z moves along world -Y -->
+    <limit lower="0.0" upper="4.5" effort="1000.0" velocity="1.0"/>
+    <!-- The origin of the platform relative to the track's slider center -->
+    <origin xyz="0 0.25 0" rpy="0 0 0"/>
   </joint>
   <!-- Mount the robot's base_mesh to the platform -->
@@ -94,5 +94,5 @@
     <parent link="world"/>
     <child link="target_panel"/>
-    <origin xyz="1.1 -4.85 1.0" rpy="0 0 0"/>
+    <origin xyz="1.5 -2.25 1.0" rpy="0 0 0"/>
   </joint>
   <!-- Load robot -->

Commit message: fix: Re-apply 180-degree rail flip to hide cables, but properly center track at world origin and correctly position the 4x2m curved surface panel

File: ros2_ws/src/irb2600_description/urdf/irb2600.urdf.xacro (robot description, xacro)
@@ -56,5 +56,6 @@
     <parent link="world"/>
     <child link="track_link"/>
-    <origin xyz="0 0 0" rpy="1.5708 0 0"/>
+    <!-- Rotate 180 around Z to put cables on the back. Shift Y by -4.3 to center the 8.6m track at world origin -->
+    <origin xyz="0 -4.3 0" rpy="1.5708 0 3.14159265359"/>
   </joint>
   <!-- Prismatic joint for the linear track -->
@@ -94,5 +95,5 @@
     <parent link="world"/>
     <child link="target_panel"/>
-    <origin xyz="1.5 -2.25 1.0" rpy="0 0 0"/>
+    <origin xyz="0.2 -2.05 1.0" rpy="0 0 0"/>
   </joint>
   <!-- Load robot -->

Commit message: fix: Replace hardcoded tank.stl with curved_panel.stl in URDF visual and collision nodes so RViz renders the correct surface

File: ros2_ws/src/irb2600_description/urdf/irb2600.urdf.xacro (robot description, xacro)
@@ -78,5 +78,5 @@
       <origin xyz="0 0 0" rpy="0 0 0"/>
       <geometry>
-        <mesh filename="package://irb2600_coating_cell/meshes/tank.stl"/>
+        <mesh filename="package://irb2600_coating_cell/meshes/curved_panel.stl"/>
       </geometry>
       <material name="panel_white">
@@ -87,5 +87,5 @@
       <origin xyz="0 0 0" rpy="0 0 0"/>
       <geometry>
-        <mesh filename="package://irb2600_coating_cell/meshes/tank.stl"/>
+        <mesh filename="package://irb2600_coating_cell/meshes/curved_panel.stl"/>
       </geometry>
     </collision>

Commit message: fix: Adjust panel position and standoff distance to avoid MoveIt collision and singularity failures

File: ros2_ws/src/irb2600_description/urdf/irb2600.urdf.xacro (robot description, xacro)
@@ -95,5 +95,5 @@
     <parent link="world"/>
     <child link="target_panel"/>
-    <origin xyz="0.2 -2.05 1.0" rpy="0 0 0"/>
+    <origin xyz="0.6 -2.05 1.0" rpy="0 0 0"/>
   </joint>
   <!-- Load robot -->

Commit message: fix: Center panel in reachable workspace and correct robot pedestal alignment after track flip

File: ros2_ws/src/irb2600_description/urdf/irb2600.urdf.xacro (robot description, xacro)
@@ -92,8 +92,8 @@
   </link>
   <!-- Mount target panel to world at the center of the track reach -->
-  <joint name="world_to_panel" type="fixed">
+  <joint name="world_to_target_panel" type="fixed">
     <parent link="world"/>
     <child link="target_panel"/>
-    <origin xyz="0.6 -2.05 1.0" rpy="0 0 0"/>
+    <origin xyz="0.6 -0.55 1.0" rpy="0 0 0"/>
   </joint>
   <!-- Load robot -->

File: ros2_ws/src/irb2600_description/urdf/robot_base.xacro (robot description, xacro)
@@ -28,11 +28,12 @@
     <parent link="platform_link"/>
     <child link="base_mesh"/>
-    <!-- Add 180 yaw (-3.14159) to keep robot facing World +X despite platform rotation -->
-    <origin xyz="0.65 0.6 1.5" rpy="1.5708 0 3.14159265359"/>
+    <!-- Use original RPY so pedestal perfectly mounts on the carriage hole -->
+    <origin xyz="0.65 0.6 1.5" rpy="-1.5708 0 0"/>
   </joint>
   <joint name="base_robot_joint" type="fixed">
     <parent link="base_mesh"/>
     <child link="base_link"/>
-    <origin xyz="0 0 0.378" rpy="0 0 0"/>
+    <!-- Add 180 yaw here to spin the arm 180 degrees in place, so it faces +X -->
+    <origin xyz="0 0 0.378" rpy="0 0 3.14159265359"/>
   </joint>
 </robot>

Commit message: fix: Exact carriage track alignment and pedestal Z offset fixes

File: ros2_ws/src/irb2600_description/urdf/irb2600.urdf.xacro (robot description, xacro)
@@ -63,15 +63,11 @@
     <parent link="track_link"/>
     <child link="platform_link"/>
-    <!-- The STL's Z-axis corresponds to the length of the track -->
+    <!-- Center the carriage on the track rails -->
+    <origin xyz="-0.0725 0.25 0" rpy="0 0 0"/>
     <axis xyz="0 0 1"/>
     <!-- The physical track limits. Since we rotated it, +Z moves along world -Y -->
     <limit lower="0.0" upper="4.5" effort="1000.0" velocity="1.0"/>
-    <!-- The origin of the platform relative to the track's slider center -->
-    <origin xyz="0 0.25 0" rpy="0 0 0"/>
   </joint>
-  <!-- Mount the robot's base_mesh to the platform -->
-  <!-- In robot_base.xacro, base_mesh attaches to 'world'. We will change that file later so it attaches to 'platform_link'. -->
-  <!-- Or we can just not include robot_base.xacro and do it here? robot_base.xacro has base_mesh_joint. -->
-  <!-- Hardcoded Target Panel for guaranteed visibility in RViz without DDS issues -->
+  <!-- Load target panel mesh -->
   <link name="target_panel">
     <visual>
@@ -80,6 +76,6 @@
         <mesh filename="package://irb2600_coating_cell/meshes/curved_panel.stl"/>
       </geometry>
-      <material name="panel_white">
-        <color rgba="1.0 1.0 1.0 1.0"/>
+      <material name="panel_grey">
+        <color rgba="0.8 0.8 0.8 1.0"/>
       </material>
     </visual>
@@ -95,5 +91,5 @@
     <parent link="world"/>
     <child link="target_panel"/>
-    <origin xyz="0.6 -0.55 1.0" rpy="0 0 0"/>
+    <origin xyz="0.6 -1.2 1.0" rpy="0 0 0"/>
   </joint>
   <!-- Load robot -->

Commit message: fix: Align platform blocks to encase track rails

File: ros2_ws/src/irb2600_description/urdf/irb2600.urdf.xacro (robot description, xacro)
@@ -63,6 +63,6 @@
     <parent link="track_link"/>
     <child link="platform_link"/>
-    <!-- Center the carriage on the track rails -->
-    <origin xyz="-0.0725 0.25 0" rpy="0 0 0"/>
+    <!-- Align sliding blocks (X=-0.064) and seat grooves on rails (Y=0.100) -->
+    <origin xyz="-0.064 0.10 0" rpy="0 0 0"/>
     <axis xyz="0 0 1"/>
     <!-- The physical track limits. Since we rotated it, +Z moves along world -Y -->

Commit message: fix: Manual tune for track sliding block visual offset

File: ros2_ws/src/irb2600_description/urdf/irb2600.urdf.xacro (robot description, xacro)
@@ -63,6 +63,8 @@
     <parent link="track_link"/>
     <child link="platform_link"/>
-    <!-- Align sliding blocks (X=-0.064) and seat grooves on rails (Y=0.100) -->
-    <origin xyz="-0.064 0.10 0" rpy="0 0 0"/>
+    <!-- Ajuste manual de encaje:
+         - X mueve la plataforma izquierda/derecha. Modificar para alinear la abertura con el riel.
+         - Y mueve la plataforma arriba/abajo. Modificar para incrustar la abertura en el riel. -->
+    <origin xyz="-0.130 0.05 0" rpy="0 0 0"/>
     <axis xyz="0 0 1"/>
     <!-- The physical track limits. Since we rotated it, +Z moves along world -Y -->
