Commit message: feat: Add tune_x and tune_y joints for live RViz tuning

File: ros2_ws/src/irb2600_description/urdf/irb2600.urdf.xacro (robot description, xacro)
@@ -59,12 +59,27 @@
     <origin xyz="0 -4.3 0" rpy="1.5708 0 3.14159265359"/>
   </joint>
+  <!-- ENLACES TEMPORALES PARA AJUSTE EN RVIZ -->
+  <link name="tune_x_link"/>
+  <link name="tune_y_link"/>
+  <joint name="tune_x_joint" type="prismatic">
+    <parent link="track_link"/>
+    <child link="tune_x_link"/>
+    <origin xyz="0 0 0" rpy="0 0 0"/>
+    <axis xyz="1 0 0"/>
+    <limit lower="-0.5" upper="0.5" effort="10" velocity="1"/>
+  </joint>
+  <joint name="tune_y_joint" type="prismatic">
+    <parent link="tune_x_link"/>
+    <child link="tune_y_link"/>
+    <origin xyz="0 0 0" rpy="0 0 0"/>
+    <axis xyz="0 1 0"/>
+    <limit lower="-0.5" upper="0.5" effort="10" velocity="1"/>
+  </joint>
   <!-- Prismatic joint for the linear track -->
   <joint name="track_prismatic_joint" type="prismatic">
-    <parent link="track_link"/>
+    <parent link="tune_y_link"/>
     <child link="platform_link"/>
-    <!-- Ajuste manual de encaje:
-         - X mueve la plataforma izquierda/derecha. Modificar para alinear la abertura con el riel.
-         - Y mueve la plataforma arriba/abajo. Modificar para incrustar la abertura en el riel. -->
-    <origin xyz="-0.130 0.05 0" rpy="0 0 0"/>
+    <!-- Origen en 0 porque los sliders de X y Y harán todo el trabajo -->
+    <origin xyz="0 0 0" rpy="0 0 0"/>
     <axis xyz="0 0 1"/>
     <!-- The physical track limits. Since we rotated it, +Z moves along world -Y -->

Commit message: fix: Lock in visual track offset and move panel closer to robot to avoid reachability limits

File: ros2_ws/src/irb2600_description/urdf/irb2600.urdf.xacro (robot description, xacro)
@@ -59,27 +59,10 @@
     <origin xyz="0 -4.3 0" rpy="1.5708 0 3.14159265359"/>
   </joint>
-  <!-- ENLACES TEMPORALES PARA AJUSTE EN RVIZ -->
-  <link name="tune_x_link"/>
-  <link name="tune_y_link"/>
-  <joint name="tune_x_joint" type="prismatic">
-    <parent link="track_link"/>
-    <child link="tune_x_link"/>
-    <origin xyz="0 0 0" rpy="0 0 0"/>
-    <axis xyz="1 0 0"/>
-    <limit lower="-0.5" upper="0.5" effort="10" velocity="1"/>
-  </joint>
-  <joint name="tune_y_joint" type="prismatic">
-    <parent link="tune_x_link"/>
-    <child link="tune_y_link"/>
-    <origin xyz="0 0 0" rpy="0 0 0"/>
-    <axis xyz="0 1 0"/>
-    <limit lower="-0.5" upper="0.5" effort="10" velocity="1"/>
-  </joint>
   <!-- Prismatic joint for the linear track -->
   <joint name="track_prismatic_joint" type="prismatic">
-    <parent link="tune_y_link"/>
+    <parent link="track_link"/>
     <child link="platform_link"/>
-    <!-- Origen en 0 porque los sliders de X y Y harán todo el trabajo -->
-    <origin xyz="0 0 0" rpy="0 0 0"/>
+    <!-- Valores precisos sintonizados visualmente por el usuario en RViz -->
+    <origin xyz="0.084 0.035 0" rpy="0 0 0"/>
     <axis xyz="0 0 1"/>
     <!-- The physical track limits. Since we rotated it, +Z moves along world -Y -->
@@ -104,9 +87,9 @@
     </collision>
   </link>
-  <!-- Mount target panel to world at the center of the track reach -->
+  <!-- Mount target panel to world at the center of the track reach, moved closer to X=0.0 to prevent reach limit errors -->
   <joint name="world_to_target_panel" type="fixed">
     <parent link="world"/>
     <child link="target_panel"/>
-    <origin xyz="0.6 -1.2 1.0" rpy="0 0 0"/>
+    <origin xyz="0.0 -1.2 1.0" rpy="0 0 0"/>
   </joint>
   <!-- Load robot -->

Commit message: feat: Add multiple passes to GUI and elevate panel. Fix GUI import error.

File: ros2_ws/src/irb2600_description/urdf/irb2600.urdf.xacro (robot description, xacro)
@@ -91,5 +91,5 @@
     <parent link="world"/>
     <child link="target_panel"/>
-    <origin xyz="0.0 -1.2 1.0" rpy="0 0 0"/>
+    <origin xyz="0.0 -1.2 1.5" rpy="0 0 0"/>
   </joint>
   <!-- Load robot -->

Commit message: feat: offset marker arrows, box collisions for track, increase raster res

File: ros2_ws/src/irb2600_description/urdf/irb2600.urdf.xacro (robot description, xacro)
@@ -18,7 +18,8 @@
     </visual>
     <collision>
-      <origin xyz="0 0 0" rpy="0 0 0"/>
+      <!-- Centered around the origin of the track link. Length is 8.6m along Z axis -->
+      <origin xyz="0 0.15 4.3" rpy="0 0 0"/>
       <geometry>
-        <mesh filename="package://irb2600_coating_cell/meshes/Riel.stl" scale="0.001 0.001 0.001"/>
+        <box size="1.0 0.5 8.6"/>
       </geometry>
     </collision>
@@ -38,7 +39,7 @@
     </visual>
     <collision>
-      <origin xyz="0 0 0" rpy="0 0 0"/>
+      <origin xyz="0 0 0.1" rpy="0 0 0"/>
       <geometry>
-        <mesh filename="package://irb2600_coating_cell/meshes/PlataformaRiel.STL" scale="0.001 0.001 0.001"/>
+        <box size="0.9 0.9 0.2"/>
       </geometry>
     </collision>
@@ -69,28 +70,4 @@
     <limit lower="0.0" upper="4.5" effort="1000.0" velocity="1.0"/>
   </joint>
-  <!-- Load target panel mesh -->
-  <link name="target_panel">
-    <visual>
-      <origin xyz="0 0 0" rpy="0 0 0"/>
-      <geometry>
-        <mesh filename="package://irb2600_coating_cell/meshes/curved_panel.stl"/>
-      </geometry>
-      <material name="panel_grey">
-        <color rgba="0.8 0.8 0.8 1.0"/>
-      </material>
-    </visual>
-    <collision>
-      <origin xyz="0 0 0" rpy="0 0 0"/>
-      <geometry>
-        <mesh filename="package://irb2600_coating_cell/meshes/curved_panel.stl"/>
-      </geometry>
-    </collision>
-  </link>
-  <!-- Mount target panel to world at the center of the track reach, moved closer to X=0.0 to prevent reach limit errors -->
-  <joint name="world_to_target_panel" type="fixed">
-    <parent link="world"/>
-    <child link="target_panel"/>
-    <origin xyz="0.0 -1.2 1.5" rpy="0 0 0"/>
-  </joint>
   <!-- Load robot -->
   <xacro:abb_irb2600 prefix=""/>

Commit message: fix: restore visual panel and use standard RViz interactive arrows

File: ros2_ws/src/irb2600_description/urdf/irb2600.urdf.xacro (robot description, xacro)
@@ -70,4 +70,23 @@
     <limit lower="0.0" upper="4.5" effort="1000.0" velocity="1.0"/>
   </joint>
+  <!-- Load target panel visual mesh so it renders beautifully in RViz -->
+  <link name="target_panel">
+    <visual>
+      <origin xyz="0 0 0" rpy="0 0 0"/>
+      <geometry>
+        <mesh filename="package://irb2600_coating_cell/meshes/curved_panel.stl"/>
+      </geometry>
+      <material name="panel_grey">
+        <color rgba="0.8 0.8 0.8 1.0"/>
+      </material>
+    </visual>
+    <!-- No <collision> tag here! The collision is handled dynamically by scene_setup_node.py -->
+  </link>
+  <!-- Mount target panel visual to world (using the correct offset where the panel physically sits) -->
+  <joint name="world_to_target_panel" type="fixed">
+    <parent link="world"/>
+    <child link="target_panel"/>
+    <origin xyz="1.5 -1.2 1.5" rpy="0 0 0"/>
+  </joint>
   <!-- Load robot -->
   <xacro:abb_irb2600 prefix=""/>

Commit message: feat: move entire scene closer to robot by 0.3m for better reachability

File: ros2_ws/src/irb2600_description/urdf/irb2600.urdf.xacro (robot description, xacro)
@@ -87,5 +87,5 @@
     <parent link="world"/>
     <child link="target_panel"/>
-    <origin xyz="1.5 -1.2 1.5" rpy="0 0 0"/>
+    <origin xyz="1.2 -1.2 1.5" rpy="0 0 0"/>
   </joint>
   <!-- Load robot -->

Commit message: feat: move scene even closer so obstacles visually touch the curved panel edges

File: ros2_ws/src/irb2600_description/urdf/irb2600.urdf.xacro (robot description, xacro)
@@ -87,5 +87,5 @@
     <parent link="world"/>
     <child link="target_panel"/>
-    <origin xyz="1.2 -1.2 1.5" rpy="0 0 0"/>
+    <origin xyz="1.0 -1.2 1.5" rpy="0 0 0"/>
   </joint>
   <!-- Load robot -->

Commit message: fix: move target canvas closer to track to prevent out-of-reach Cartesian path failures

File: ros2_ws/src/irb2600_description/urdf/irb2600.urdf.xacro (robot description, xacro)
@@ -87,5 +87,5 @@
     <parent link="world"/>
     <child link="target_panel"/>
-    <origin xyz="1.0 -1.2 1.5" rpy="0 0 0"/>
+    <origin xyz="0.75 -1.2 1.5" rpy="0 0 0"/>
   </joint>
   <!-- Load robot -->

Commit message: fix: fine-tune canvas distance to 0.9m to avoid self-collisions and allow bypass on failed cartesian path

File: ros2_ws/src/irb2600_description/urdf/irb2600.urdf.xacro (robot description, xacro)
@@ -87,5 +87,5 @@
     <parent link="world"/>
     <child link="target_panel"/>
-    <origin xyz="0.75 -1.2 1.5" rpy="0 0 0"/>
+    <origin xyz="0.9 -1.2 1.5" rpy="0 0 0"/>
   </joint>
   <!-- Load robot -->

Commit message: fix: aggressively move canvas to 0.5m to maximize manipulability and prevent KDL kinematics failures

File: ros2_ws/src/irb2600_description/urdf/irb2600.urdf.xacro (robot description, xacro)
@@ -87,5 +87,5 @@
     <parent link="world"/>
     <child link="target_panel"/>
-    <origin xyz="0.9 -1.2 1.5" rpy="0 0 0"/>
+    <origin xyz="0.5 -1.2 1.5" rpy="0 0 0"/>
   </joint>
   <!-- Load robot -->

Commit message: fix: set canvas to 0.85m to allow RRT bypass space, and increase KDL timeout to 0.5s to prevent Cartesian failures

File: ros2_ws/src/irb2600_description/urdf/irb2600.urdf.xacro (robot description, xacro)
@@ -87,5 +87,5 @@
     <parent link="world"/>
     <child link="target_panel"/>
-    <origin xyz="0.5 -1.2 1.5" rpy="0 0 0"/>
+    <origin xyz="0.85 -1.2 1.5" rpy="0 0 0"/>
   </joint>
   <!-- Load robot -->

Commit message: fix: remove canvas from collision scene to allow RRT bypass jumps while keeping canvas at optimal 0.5m for Cartesian paths

File: ros2_ws/src/irb2600_description/urdf/irb2600.urdf.xacro (robot description, xacro)
@@ -87,5 +87,5 @@
     <parent link="world"/>
     <child link="target_panel"/>
-    <origin xyz="0.85 -1.2 1.5" rpy="0 0 0"/>
+    <origin xyz="0.5 -1.2 1.5" rpy="0 0 0"/>
   </joint>
   <!-- Load robot -->

Commit message: fix: re-enable canvas collision and set to 0.7m to balance RRT clearance and KDL track dragging

File: ros2_ws/src/irb2600_description/urdf/irb2600.urdf.xacro (robot description, xacro)
@@ -87,5 +87,5 @@
     <parent link="world"/>
     <child link="target_panel"/>
-    <origin xyz="0.5 -1.2 1.5" rpy="0 0 0"/>
+    <origin xyz="0.7 -1.2 1.5" rpy="0 0 0"/>
   </joint>
   <!-- Load robot -->

Commit message: fix: fine-tune canvas to 0.6m and constrain arm posture to prevent orientation flips

File: ros2_ws/src/irb2600_description/urdf/irb2600.urdf.xacro (robot description, xacro)
@@ -87,5 +87,5 @@
     <parent link="world"/>
     <child link="target_panel"/>
-    <origin xyz="0.7 -1.2 1.5" rpy="0 0 0"/>
+    <origin xyz="0.6 -1.2 1.5" rpy="0 0 0"/>
   </joint>
   <!-- Load robot -->

Commit message: cambios v2

File: ros2_ws/src/irb2600_description/urdf/irb2600.urdf.xacro (robot description, xacro)
@@ -70,23 +70,7 @@
     <limit lower="0.0" upper="4.5" effort="1000.0" velocity="1.0"/>
   </joint>
-  <!-- Load target panel visual mesh so it renders beautifully in RViz -->
-  <link name="target_panel">
-    <visual>
-      <origin xyz="0 0 0" rpy="0 0 0"/>
-      <geometry>
-        <mesh filename="package://irb2600_coating_cell/meshes/curved_panel.stl"/>
-      </geometry>
-      <material name="panel_grey">
-        <color rgba="0.8 0.8 0.8 1.0"/>
-      </material>
-    </visual>
-    <!-- No <collision> tag here! The collision is handled dynamically by scene_setup_node.py -->
-  </link>
-  <!-- Mount target panel visual to world (using the correct offset where the panel physically sits) -->
-  <joint name="world_to_target_panel" type="fixed">
-    <parent link="world"/>
-    <child link="target_panel"/>
-    <origin xyz="0.6 -1.2 1.5" rpy="0 0 0"/>
-  </joint>
+  <!-- The panel is visualized and collision-checked by scene_setup_node.
+       Keeping it out of this static URDF ensures an observed 6D panel pose
+       cannot be rendered twice at conflicting locations. -->
   <!-- Load robot -->
   <xacro:abb_irb2600 prefix=""/>

File: ros2_ws/src/irb2600_description/urdf/spray_nozzle.xacro (robot description, xacro)
@@ -2,8 +2,8 @@
 <robot xmlns:xacro="http://ros.org/wiki/xacro">
   <!--
-    Simulated spraying-nozzle end effector (report Table V/VIII: "Spraying nozzle
-    (simulated)"). Geometry is reused from RAMEL-ESPOL/IRB2600-ABB
-    irb2600_description/urdf/ee_marker.xacro (the whiteboard-marker tool), which is
-    a reasonable placeholder standoff length until a real nozzle CAD is available.
+    Cobra spraying-nozzle end effector.  Its visual mesh comes from the
+    supplied Cobra CAD export.  The collision geometry is deliberately a
+    conservative box derived from that export's bounds, so MoveIt does not
+    need to process the 119k-triangle presentation mesh on every plan.
     Frames:
       tool0            - ROS-Industrial flange-facing frame (from irb2600_macro.xacro)
@@ -40,7 +40,10 @@
     </visual>
     <collision>
-      <origin xyz="0 0 0" rpy="0 0 0"/>
+      <!-- CobraPaintTool STL bounds, converted from mm to m:
+           342.479 x 100.750 x 88.713.  Offset is its bounding-box center
+           in the source mesh frame. -->
+      <origin xyz="0.174107 0.056650 0.054678" rpy="0 0 0"/>
       <geometry>
-        <mesh filename="package://irb2600_coating_cell/meshes/CobraPaintTool.STL" scale="0.001 0.001 0.001"/>
+        <box size="0.342479 0.100750 0.088713"/>
       </geometry>
     </collision>
