Commit message: fix: Align spray nozzle to flange, fix default target position in executor, and add panel to collision objects for RViz visualization

File: ros2_ws/src/irb2600_description/urdf/spray_nozzle.xacro (robot description, xacro)
@@ -49,5 +49,6 @@
     <parent link="tool0"/>
     <child link="spray_nozzle_link"/>
-    <origin xyz="0 0 0" rpy="1.57 0 0"/>
+    <!-- CobraPaintTool length is along its X axis. We pitch by -90 deg to align it with tool0's Z axis (outward). -->
+    <origin xyz="0 0 0" rpy="0 -1.5708 0"/>
   </joint>
   <!-- TCP: x_e in the preliminary mathematical model (report eq. 1-2, 8-9) -->
@@ -61,5 +62,5 @@
   </link>
   <joint name="tool0_to_nozzle_tip" type="fixed">
-    <origin xyz="0 0 0.14" rpy="0 0 0"/>
+    <origin xyz="0 0 0.35" rpy="0 0 0"/>
     <parent link="tool0"/>
     <child link="nozzle_tip"/>

Commit message: fix: Center panel perfectly at Y=-4.0 within track limits

File: ros2_ws/src/irb2600_description/urdf/spray_nozzle.xacro (robot description, xacro)
@@ -49,6 +49,7 @@
     <parent link="tool0"/>
     <child link="spray_nozzle_link"/>
-    <!-- CobraPaintTool length is along its X axis. We pitch by -90 deg to align it with tool0's Z axis (outward). -->
-    <origin xyz="0 0 0" rpy="0 -1.5708 0"/>
+    <!-- CobraPaintTool length is along its X axis, and its mounting plate center is offset in Y and Z.
+         We pitch by -90 deg to align X with tool0's Z axis (outward), and offset XYZ to center it on the flange. -->
+    <origin xyz="0.054 -0.056 0" rpy="0 -1.5708 0"/>
   </joint>
   <!-- TCP: x_e in the preliminary mathematical model (report eq. 1-2, 8-9) -->

Commit message: feat: add 14cm collision cylinder to nozzle_tip to model spray paint volume and force MoveIt to avoid spraying over obstacles

File: ros2_ws/src/irb2600_description/urdf/spray_nozzle.xacro (robot description, xacro)
@@ -61,4 +61,11 @@
       </geometry>
     </visual>
+    <!-- 14cm collision cylinder representing the paint spray. This forces MoveIt to dodge obstacles that block the spray path, rather than just obstacles that hit the physical arm. -->
+    <collision>
+      <origin xyz="0 0 0.07" rpy="0 0 0"/>
+      <geometry>
+        <cylinder radius="0.05" length="0.14"/>
+      </geometry>
+    </collision>
   </link>
   <joint name="tool0_to_nozzle_tip" type="fixed">

Commit message: revert: remove spray collision volume that was causing path planning failures on the normal route

File: ros2_ws/src/irb2600_description/urdf/spray_nozzle.xacro (robot description, xacro)
@@ -61,11 +61,4 @@
       </geometry>
     </visual>
-    <!-- 14cm collision cylinder representing the paint spray. This forces MoveIt to dodge obstacles that block the spray path, rather than just obstacles that hit the physical arm. -->
-    <collision>
-      <origin xyz="0 0 0.07" rpy="0 0 0"/>
-      <geometry>
-        <cylinder radius="0.05" length="0.14"/>
-      </geometry>
-    </collision>
   </link>
   <joint name="tool0_to_nozzle_tip" type="fixed">

Commit message: correccion del brazo v1

File: ros2_ws/src/irb2600_description/urdf/spray_nozzle.xacro (robot description, xacro)
@@ -54,12 +54,6 @@
   </joint>
   <!-- TCP: x_e in the preliminary mathematical model (report eq. 1-2, 8-9) -->
-  <link name="nozzle_tip">
-    <visual>
-      <origin xyz="0 0 0" rpy="0 0 0"/>
-      <geometry>
-        <box size="0.01 0.01 0.01"/>
-      </geometry>
-    </visual>
-  </link>
+  <!-- Coordinate-only link: deliberately has no visual/collision geometry. -->
+  <link name="nozzle_tip"/>
   <joint name="tool0_to_nozzle_tip" type="fixed">
     <origin xyz="0 0 0.35" rpy="0 0 0"/>

Commit message: cambios v3

File: ros2_ws/src/irb2600_description/urdf/spray_nozzle.xacro (robot description, xacro)
@@ -5,5 +5,5 @@
     supplied Cobra CAD export.  The collision geometry is deliberately a
     conservative box derived from that export's bounds, so MoveIt does not
-    need to process the 119k-triangle presentation mesh on every plan.
+    need to process the high-detail presentation mesh on every plan.
     Frames:
       tool0            - ROS-Industrial flange-facing frame (from irb2600_macro.xacro)
@@ -24,4 +24,10 @@
     material_abb_orange macro, assuming it is already defined.
   -->
+  <!-- Calibration inputs. Defaults preserve the prior digital model; replace
+       them with the measured tool0-to-Cobra and tool0-to-TCP transforms. -->
+  <xacro:arg name="cobra_mount_xyz" default="0.054 -0.056 0"/>
+  <xacro:arg name="cobra_mount_rpy" default="0 -1.5708 0"/>
+  <xacro:arg name="cobra_tcp_xyz" default="0 0 0.35"/>
+  <xacro:arg name="cobra_tcp_rpy" default="0 0 0"/>
   <link name="spray_nozzle_link">
     <inertial>
@@ -35,15 +41,15 @@
       <origin xyz="0 0 0" rpy="0 0 0"/>
       <geometry>
-        <mesh filename="package://irb2600_coating_cell/meshes/CobraPaintTool.STL" scale="0.001 0.001 0.001"/>
+        <mesh filename="package://irb2600_coating_cell/meshes/cad/cobra_final.stl"/>
       </geometry>
       <xacro:material_abb_orange/>
     </visual>
     <collision>
-      <!-- CobraPaintTool STL bounds, converted from mm to m:
-           342.479 x 100.750 x 88.713.  Offset is its bounding-box center
-           in the source mesh frame. -->
-      <origin xyz="0.174107 0.056650 0.054678" rpy="0 0 0"/>
+      <!-- Final Cobra assembly STL bounds in metres:
+           342.479 x 315.413 x 108.000. The box center is expressed in the
+           STL frame and envelopes the complete assembly. -->
+      <origin xyz="-0.115471 -0.122706 0.0" rpy="0 0 0"/>
       <geometry>
-        <box size="0.342479 0.100750 0.088713"/>
+        <box size="0.342479 0.315413 0.108000"/>
       </geometry>
     </collision>
@@ -52,7 +58,6 @@
     <parent link="tool0"/>
     <child link="spray_nozzle_link"/>
-    <!-- CobraPaintTool length is along its X axis, and its mounting plate center is offset in Y and Z.
-         We pitch by -90 deg to align X with tool0's Z axis (outward), and offset XYZ to center it on the flange. -->
-    <origin xyz="0.054 -0.056 0" rpy="0 -1.5708 0"/>
+    <!-- Provisional calibration; replace with the measured mounting transform. -->
+    <origin xyz="$(arg cobra_mount_xyz)" rpy="$(arg cobra_mount_rpy)"/>
   </joint>
   <!-- TCP: x_e in the preliminary mathematical model (report eq. 1-2, 8-9) -->
@@ -60,5 +65,5 @@
   <link name="nozzle_tip"/>
   <joint name="tool0_to_nozzle_tip" type="fixed">
-    <origin xyz="0 0 0.35" rpy="0 0 0"/>
+    <origin xyz="$(arg cobra_tcp_xyz)" rpy="$(arg cobra_tcp_rpy)"/>
     <parent link="tool0"/>
     <child link="nozzle_tip"/>
